Commit message: Updated readme

File: src/mybot_description/urdf/mybot.xacro (robot description, xacro)
@@ -27,4 +27,5 @@
         <box size=".4 .2 .1"/>
       </geometry>
+      <material name="orange"/>
     </visual>
     <collision name='caster_collision'>
@@ -50,4 +51,5 @@
       </geometry>
     </visual>
+      <material name="grey"/>
   </link>
   <link name="left_wheel">
@@ -64,4 +66,5 @@
         <cylinder radius="0.1" length="0.05"/>
       </geometry>
+	<material name="grey"/>
     </visual>
     <inertial>
@@ -88,4 +91,5 @@
         <cylinder radius="0.1" length="0.05"/>
       </geometry>
+	<material name="grey"/>
     </visual>
     <inertial>

Commit message: added navigation, updated readme

File: src/mybot_description/urdf/mybot.xacro (robot description, xacro)
@@ -9,9 +9,9 @@
     <pose>0 0 0.1 0 0 0</pose>
     <inertial>
-      <mass value="10.0"/>
+      <mass value="15.0"/>
       <origin xyz="0.0 0 0.1" rpy=" 0 0 0"/>
       <inertia
-          ixx="0.5" ixy="0" ixz="0"
-          iyy="1.0" iyz="0"
+          ixx="0.1" ixy="0" ixz="0"
+          iyy="0.1" iyz="0"
           izz="0.1"
       />
@@ -50,6 +50,28 @@
         <sphere radius="0.05"/>
       </geometry>
+      <material name="grey"/>
     </visual>
-      <material name="grey"/>
+    <collision name='caster_front_collision'>
+      <origin xyz="0.15 0 -0.05" rpy=" 0 0 0"/>
+      <geometry>
+        <sphere radius="0.05"/>
+      </geometry>
+      <surface>
+        <friction>
+          <ode>
+            <mu>0</mu>
+            <mu2>0</mu2>
+            <slip1>1.0</slip1>
+            <slip2>1.0</slip2>
+          </ode>
+        </friction>
+      </surface>
+    </collision>
+    <visual name='caster_front_visual'>
+      <origin xyz="0.15 0 -0.05" rpy=" 0 0 0"/>
+      <geometry>
+        <sphere radius="0.05"/>
+      </geometry>
+    </visual>
   </link>
   <link name="left_wheel">
@@ -71,9 +93,8 @@
       <origin xyz="0 0 0" rpy="0 1.5707 1.5707"/>
       <mass value="5"/>
-      <cylinder_inertia m="5" r="0.1" h="0.05"/>
       <inertia
-        ixx="1.0" ixy="0.0" ixz="0.0"
-        iyy="1.0" iyz="0.0"
-        izz="1.0"/>
+        ixx=".1" ixy="0.0" ixz="0.0"
+        iyy=".1" iyz="0.0"
+        izz=".1"/>
     </inertial>
   </link>
@@ -96,28 +117,29 @@
       <origin xyz="0 0 0" rpy="0 1.5707 1.5707"/>
       <mass value="5"/>
-      <cylinder_inertia m="5" r="0.1" h="0.05"/>
       <inertia
-        ixx="1.0" ixy="0.0" ixz="0.0"
-        iyy="1.0" iyz="0.0"
-        izz="1.0"/>
+        ixx=".1" ixy="0.0" ixz="0.0"
+        iyy=".1" iyz="0.0"
+        izz=".1"/>
     </inertial>
   </link>
   <joint type="continuous" name="left_wheel_hinge">
-    <origin xyz="0.1 0.15 0" rpy="0 0 0"/>
+    <origin xyz="0 0.15 0" rpy="0 0 0"/>
+    <!--origin xyz="0.1 0.13 0" rpy="0 1.5707 1.5707"/-->
     <child link="left_wheel"/>
     <parent link="chassis"/>
     <axis xyz="0 1 0" rpy="0 0 0"/>
-    <limit effort="100" velocity="100"/>
-    <joint_properties damping="0.0" friction="0.0"/>
+    <limit effort="10000" velocity="1000"/>
+    <joint_properties damping="1.0" friction="1.0"/>
   </joint>
   <joint type="continuous" name="right_wheel_hinge">
-    <origin xyz="0.1 -0.15 0" rpy="0 0 0"/>
+    <origin xyz="0 -0.15 0" rpy="0 0 0"/>
+    <!--origin xyz="0.1 -0.13 0" rpy="0 1.5707 1.5707"/-->
     <child link="right_wheel"/>
     <parent link="chassis"/>
     <axis xyz="0 1 0" rpy="0 0 0"/>
-    <limit effort="100" velocity="100"/>
-    <joint_properties damping="0.0" friction="0.0"/>
+    <limit effort="10000" velocity="1000"/>
+    <joint_properties damping="1.0" friction="1.0"/>
   </joint>
-<link name="camera">
+  <link name="camera">
     <collision>
       <origin xyz="0 0 0" rpy="0 0 0"/>
@@ -146,4 +168,10 @@
     <child link="camera"/>
   </joint>
+  <joint name="hokuyo_joint" type="fixed">
+    <axis xyz="0 1 0" />
+    <origin xyz=".15 0 .1" rpy="0 0 0"/>
+    <parent link="chassis"/>
+    <child link="hokuyo"/>
+  </joint>
   <!-- Hokuyo Laser -->
   <link name="hokuyo">
@@ -165,10 +193,4 @@
       <inertia ixx="1e-6" ixy="0" ixz="0" iyy="1e-6" iyz="0" izz="1e-6" />
     </inertial>
-</link>
-  <joint name="hokuyo_joint" type="fixed">
-    <axis xyz="0 1 0" />
-    <origin xyz=".15 0 .1" rpy="0 0 0"/>
-    <parent link="chassis"/>
-    <child link="hokuyo"/>
-  </joint>
+  </link>
 </robot>
